File: KiCAD/Prawn/PrawnBlaster_Connectorized.kicad_pcb (KiCad board)
At the start: 2 copper layers, 93 x 58.4 mm, 37 parts, among them IC1 74LVT245D,118, J1 PWR SEL, J2 Ext. Clock, J3 Ext. Trig., J4 Pseudoclock 3, J5 Pseudoclock 1, J6 Pseudoclock 2, J7 Pseudoclock 0, J8 EXT PWR, U2 74LVC1G34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

Commit message: Corrected branches
Parts:
- moved R15 0.11 mm to (107.9, 108.1)
Routing:
- net Power Supply: track 69.0 -> 78.5 mm
- net Net-(IC1-A6): track 8.03 -> 7.00 mm
