File: KiCAD/PrawnBlaster_Connectorized.kicad_sch (KiCad schematic)
At the start: 30 parts, among them IC1 74LVT245D,118, J1 PWR SEL, J2 Ext. Clock, J3 Ext. Trig., J4 Pseudoclock 3, J5 Pseudoclock 1, J6 Pseudoclock 2, J7 Pseudoclock 0, J8 EXT PWR, U2 74LVC1G34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

Commit message: Relocate files. Make a few minor changes to the silkscreen stuff.
Parts:
- C2: value .1uF -> 1uF
Changed lines of the file:
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@@
       (effects (font (size 1.27 1.27)))
     )
-    (property "Value" ".1uF" (at 151.765 111.125 0)
+    (property "Value" "1uF" (at 151.765 111.125 0)
       (effects (font (size 1.27 1.27)))
     )
